File: stairlight_controller_pcb/stairlight_controller_pcb.kicad_sch (KiCad schematic)
At the start: 12 parts, among them J1 AC IN, J2 AC OUT, J3 DC OUT, J4 PIR_IN, K1 Relay, Q1 BC547, U1 WeMos_D1_mini

Commit message: Final Schematic and PCB
Parts:
- added R4, R5: 10K, Resistor_THT:R_Axial_DIN0204_L3.6mm_D1.6mm_P5.08mm_Horizontal, symbol Device:R
- R1: footprint OptoDevice:R_LDR_10x8.5mm_P7.6mm_Vertical -> OptoDevice:R_LDR_5.0x4.1mm_P3mm_Vertical
- R3: value 10K -> 1K
Connections:
- net GND: now also R4.1, R5.1
- net at J4.1 (Pin_1): now also U1.4 (SCK/D5), R5.2; no longer U1.5 (MISO/D6)
- net at J4.2 (Pin_2): now also U1.3 (D0), R4.2; no longer U1.4 (SCK/D5)
- net at D1.1 (K), J3.2 (Pin_2), K1.2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: no longer R1.1
- net at U1.11 (D4): no longer R2.2
- net at U1.13 (SDA/D2): now also R2.2
- net at U1.8 (3V3): now also R1.1
- no-connect marks 11 -> 10
Other:
- moved on the sheet: J4, R1, R2
